File: revisi/1phasa/untitled.brd (EAGLE design)
At the start: 80 x 80 mm, 54 parts, among them J1 U.FL-R-SMT(01), J2 10118193-0001LF, K2 SRD-05VDC-SL-C, Q1 S9013, Q16 MMBT3904, Q17 MMBT3904, Q18 12MHz, U1 AMS1117, U19 CH340G, U2 PC817X2NIP0F, U3 ESP32-WROOM-32D

Commit message: menambahkan fuse
Parts:
- added FUSE-KOTAK1: (no value), FUSE-KOTAK:FUSE-KOTAK
Connections:
- new net N$14: FUSE-KOTAK1.1, TB7.1.T2
- net N$1: now also FUSE-KOTAK1.2; no longer TB7.1.T2
Routing:
- net N$1: track 88.1 -> 78.0 mm
- net N$14: track 0.00 -> 5.29 mm
- net EN: track 141.1 -> 140.4 mm

Commit message: revisi besar-besaran
Parts:
- moved C11 0.16 mm to (59.2, 38.6)
- moved C7 0.14 mm to (57.0, 38.6)
Connections:
- net RX_PZEM: now also U3.28; no longer U3.27
- net TX_PZEM: now also U3.27; no longer U3.28
Routing:
- net TX_PZEM: track 59.5 -> 74.1 mm
- net N$7: track 34.7 -> 30.6 mm
- net GND: track 454.9 -> 451.7 mm
- net RX_PZEM: track 59.7 -> 62.8 mm
- net VCC: track 176.4 -> 178.5 mm
- net TX_SIM: track 48.0 -> 46.8 mm
- net RX_SIM: track 39.2 -> 39.9 mm
- net N$103: track 35.5 -> 36.1 mm
