File: revisi/1phasa/untitled.brd (EAGLE design)
At the start: 80 x 80 mm, 55 parts, among them J1 U.FL-R-SMT(01), J2 10118193-0001LF, K2 SRD-05VDC-SL-C, Q1 S9013, Q16 MMBT3904, Q17 MMBT3904, Q18 12MHz, U1 AMS1117, U19 CH340G, U2 PC817X2NIP0F, U3 ESP32-WROOM-32D

Commit message: revisi tanggal 05/01/2023
Other:
- board size 80 x 80 mm -> 80 x 102 mm
Changed lines of the file:
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@@
 <board>
 <plain>
-<wire x1="0" y1="80" x2="0" y2="0" width="0" layer="20"/>
-<wire x1="0" y1="0" x2="80" y2="0" width="0" layer="20"/>
-<wire x1="80" y1="0" x2="80" y2="80" width="0" layer="20"/>
-<wire x1="80" y1="80" x2="0" y2="80" width="0" layer="20"/>
+<wire x1="0" y1="91" x2="0" y2="-11" width="0" layer="20"/>
+<wire x1="0" y1="-11" x2="80" y2="-11" width="0" layer="20"/>
+<wire x1="80" y1="-11" x2="80" y2="91" width="0" layer="20"/>
+<wire x1="80" y1="91" x2="0" y2="91" width="0" layer="20"/>
 <text x="72.91520625" y="45.303959375" size="1.4224" layer="25" rot="R90">AC</text>
 <text x="72.972259375" y="59.054909375" size="1.4224" layer="25" rot="R90">CT</text>
@@
 <text x="72.92135625" y="14.94710625" size="1.4224" layer="25" rot="R90">POWER</text>
 <dimension x1="0" y1="0" x2="0" y2="80" x3="-10" y3="40" textsize="1.778" layer="1"/>
+<dimension x1="0" y1="0" x2="0" y2="-11" x3="-10" y3="-5.5" textsize="1.778" layer="1"/>
+<dimension x1="0" y1="80" x2="0" y2="91" x3="-10" y3="85.5" textsize="1.778" layer="1"/>
+<dimension x1="0" y1="91" x2="11.6" y2="91" x3="5.8" y3="94.2" textsize="1.778" layer="1"/>
 </plain>
 <attributes>

Commit message: revisi tanggal 05/01/2023
Parts:
- moved FUSE-KOTAK1 6.60 mm to (70.5, 0.15), turned to 180 degrees
- moved TB7.1 5.59 mm to (76.9, 13.2)
- moved TB7.4 5.10 mm to (77.0, 65.5)
- moved TB7.2 2.24 mm to (76.9, 30.7)
- moved TB7.3 1.80 mm to (76.9, 48.1)
Routing:
- net N$17: track 29.1 -> 35.2 mm
- net N$1: track 78.0 -> 73.4 mm
- net N$18: track 25.0 -> 20.5 mm
- net N$14: track 5.29 -> 8.97 mm
- net N$2: track 78.0 -> 74.9 mm
- net N$16: track 34.8 -> 36.0 mm
- net N$9: track 76.2 -> 77.0 mm
- net N$10: track 69.9 -> 70.7 mm
- net N$15: track 42.8 -> 43.5 mm
Other:
- outline, holes or cut-outs redrawn
Changed lines of the file:
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@@
 <setting verticaltext="up"/>
 </settings>
-<grid distance="1" unitdist="mm" unit="mm" style="lines" multiple="1" display="yes" altdistance="5" altunitdist="mil" altunit="mil"/>
+<grid distance="0.5" unitdist="mm" unit="mm" style="lines" multiple="1" display="yes" altdistance="5" altunitdist="mil" altunit="mil"/>
 <layers>
 <layer number="1" name="Top" color="4" fill="1" visible="yes" active="yes"/>
@@
 <text x="73.031809375" y="29.30210625" size="1.4224" layer="25" rot="R90">RELAY</text>
 <text x="72.92135625" y="14.94710625" size="1.4224" layer="25" rot="R90">POWER</text>
-<dimension x1="0" y1="0" x2="0" y2="80" x3="-10" y3="40" textsize="1.778" layer="1"/>
-<dimension x1="0" y1="0" x2="0" y2="-11" x3="-10" y3="-5.5" textsize="1.778" layer="1"/>
-<dimension x1="0" y1="80" x2="0" y2="91" x3="-10" y3="85.5" textsize="1.778" layer="1"/>
-<dimension x1="0" y1="91" x2="11.6" y2="91" x3="5.8" y3="94.2" textsize="1.778" layer="1"/>
+<circle x="11.6" y="87" radius="1.75" width="0.1524" layer="20"/>
+<circle x="63.2" y="-7" radius="1.75" width="0.1524" layer="20"/>
 </plain>
 <attributes>
@@
 <attribute name="VALUE" x="-2.46308125" y="68.224465625" size="1.27" layer="27" ratio="10" rot="R270"/>
 </element>
-<element name="TB7.1" library="TB7.62" package="TB7.62" value="" x="75.924909375" y="18.660603125" smashed="yes" rot="R270"/>
-<element name="TB7.2" library="TB7.62" package="TB7.62" value="" x="75.93924375" y="32.652734375" smashed="yes" rot="R270"/>
-<element name="TB7.3" library="TB7.62" package="TB7.62" value="" x="75.92705" y="46.5756125" smashed="yes" rot="R270"/>
-<element name="TB7.4" library="TB7.62" package="TB7.62" value="" x="76.00751875" y="60.530821875" smashed="yes" rot="R270"/>
+<element name="TB7.1" library="TB7.62" package="TB7.62" value="" x="76.924909375" y="13.160603125" smashed="yes" rot="R270"/>
+<element name="TB7.2" library="TB7.62" package="TB7.62" value="" x="76.93924375" y="30.652734375" smashed="yes" rot="R270"/>
+<element name="TB7.3" library="TB7.62" package="TB7.62" value="" x="76.92705" y="48.0756125" smashed="yes" rot="R270"/>
+<element name="TB7.4" library="TB7.62" package="TB7.62" value="" x="77.00751875" y="65.530821875" smashed="yes" rot="R270"/>
 <element name="U1" library="AMS1117" package="SOT229P700X180-4N" value="AMS1117" x="11.239525" y="70.6016875" smashed="yes" rot="R270">
 <attribute name="AVAILABILITY" value="Not in stock" x="-56.070475" y="24.8816875" size="1.778" layer="27" rot="R270" display="off"/>
@@
 <attribute name="VALUE" x="21.66988125" y="42.9995375" size="1.27" layer="27"/>
 </element>
-<element name="FUSE-KOTAK1" library="FUSE-KOTAK" package="FUSE-KOTAK" value="" x="75.849090625" y="3.9667375" smashed="yes" rot="R270"/>
+<element name="FUSE-KOTAK1" library="FUSE-KOTAK" package="FUSE-KOTAK" value="" x="70.4667375" y="0.150909375" smashed="yes" rot="R180"/>
 </elements>
 <signals>
@@
 <wire x1="9.065815625" y1="2.246290625" x2="7.513984375" y2="3.798121875" width="1.27" layer="16"/>
 <contactref element="FUSE-KOTAK1" pad="2"/>
-<wire x1="27.72754375" y1="2.246290625" x2="73.04864375" y2="2.246290625" width="1.27" layer="16"/>
-<wire x1="73.04864375" y1="2.246290625" x2="75.229090625" y2="4.4267375" width="1.27" layer="16"/>
+<wire x1="27.72754375" y1="2.246290625" x2="69.4095375" y2="2.246290625" width="1.27" layer="16"/>
+<wire x1="69.4095375" y1="2.246290625" x2="70.9267375" y2="0.770909375" width="1.27" layer="16"/>
 </signal>
 <signal name="N$2">
@@
 <wire x1="67.3057875" y1="5.616428125" x2="32.50131875" y2="5.616428125" width="1.27" layer="16"/>
 <wire x1="32.083403125" y1="6.03434375" x2="32.50131875" y2="5.616428125" width="1.27" layer="16"/>
-<wire x1="67.3057875" y1="5.616428125" x2="70.40483125" y2="8.715471875" width="1.27" layer="16"/>
-<wire x1="70.40483125" y1="8.715471875" x2="70.40483125" y2="19.017675" width="1.27" layer="16"/>
-<wire x1="70.40483125" y1="19.017675" x2="73.769609375" y2="22.382453125" width="1.27" layer="16"/>
-<wire x1="73.769609375" y1="22.382453125" x2="75.303059375" y2="22.382453125" width="1.27" layer="16"/>
-<wire x1="75.303059375" y1="22.382453125" x2="75.324909375" y2="22.360603125" width="1.27" layer="16"/>
+<wire x1="70.40483125" y1="8.715471875" x2="67.3057875" y2="5.616428125" width="1.27" layer="16"/>
+<wire x1="76.924909375" y1="16.960603125" x2="72.460603125" y2="16.960603125" width="1.27" layer="16"/>
+<wire x1="70.40483125" y1="14.90483125" x2="70.40483125" y2="8.715471875" width="1.27" layer="16"/>
+<wire x1="72.460603125" y1="16.960603125" x2="70.40483125" y2="14.90483125" width="1.27" layer="16"/>
 </signal>
 <signal name="N$3">
@@
 <wire x1="25.888346875" y1="23.78135" x2="30.3411625" y2="19.328534375" width="1.27" layer="16"/>
 <wire x1="30.3411625" y1="19.328534375" x2="62.722571875" y2="19.328534375" width="1.27" layer="16"/>
-<wire x1="72.146771875" y1="28.752734375" x2="75.33924375" y2="28.752734375" width="1.27" layer="16"/>
-<wire x1="62.722571875" y1="19.328534375" x2="72.146771875" y2="28.752734375" width="1.27" layer="16"/>
+<wire x1="70.12920625" y1="26.73516875" x2="76.93924375" y2="26.852734375" width="1.27" layer="16"/>
+<wire x1="62.722571875" y1="19.328534375" x2="70.12920625" y2="26.73516875" width="1.27" layer="16"/>
 </signal>
 <signal name="N$4">
@@
 <wire x1="48.654903125" y1="72.78418125" x2="49.463740625" y2="71.97534375" width="1.27" layer="16"/>
 <wire x1="49.463740625" y1="71.97534375" x2="49.463740625" y2="66.09060625" width="1.27" layer="16"/>
-<wire x1="73.11695625" y1="42.437390625" x2="75.088828125" y2="42.437390625" width="1.27" layer="16"/>
-<wire x1="49.463740625" y1="66.09060625" x2="73.11695625" y2="42.437390625" width="1.27" layer="16"/>
-<wire x1="75.32705" y1="42.6756125" x2="75.088828125" y2="42.437390625" width="1.27" layer="16"/>
+<wire x1="49.463740625" y1="66.09060625" x2="70.527171875" y2="45.027175" width="1.27" layer="16"/>
+<wire x1="76.92705" y1="44.2756125" x2="71.278734375" y2="44.2756125" width="1.27" layer="16"/>
+<wire x1="71.278734375" y1="44.2756125" x2="70.527171875" y2="45.027175" width="1.27" layer="16"/>
 </signal>
 <signal name="N$16">
 <contactref element="PZEM004T1" pad="CT1-"/>
 <contactref element="TB7.3" pad="T1"/>
-<wire x1="53.734903125" y1="72.78418125" x2="53.734903125" y2="66.28553125" width="1.27" layer="16"/>
-<wire x1="53.734903125" y1="66.28553125" x2="69.8590125" y2="50.161421875" width="1.27" layer="16"/>
-<wire x1="69.8590125" y1="50.161421875" x2="75.212859375" y2="50.161421875" width="1.27" layer="16"/>
-<wire x1="75.212859375" y1="50.161421875" x2="75.32705" y2="50.2756125" width="1.27" layer="16"/>
+<wire x1="53.734903125" y1="72.78418125" x2="53.734903125" y2="65.78553125" width="1.27" layer="16"/>
+<wire x1="76.92705" y1="51.8756125" x2="67.644821875" y2="51.8756125" width="1.27" layer="16"/>
+<wire x1="67.644821875" y1="51.8756125" x2="53.734903125" y2="65.78553125" width="1.27" layer="16"/>
 </signal>
 <signal name="N$17">
 <contactref element="PZEM004T1" pad="L1"/>
 <contactref element="TB7.4" pad="T2"/>
-<wire x1="58.814903125" y1="72.78418125" x2="58.814903125" y2="65.0179125" width="1.016" layer="16"/>
-<wire x1="58.814903125" y1="65.0179125" x2="68.68546875" y2="55.147346875" width="1.016" layer="16"/>
-<wire x1="68.68546875" y1="55.147346875" x2="73.92404375" y2="55.147346875" width="1.016" layer="16"/>
-<wire x1="73.92404375" y1="55.147346875" x2="75.40751875" y2="56.630821875" width="1.016" layer="16"/>
+<wire x1="58.814903125" y1="72.78418125" x2="58.814903125" y2="64.5179125" width="1.016" layer="16"/>
+<wire x1="58.814903125" y1="64.5179125" x2="68.538546875" y2="54.79426875" width="1.016" layer="16"/>
+<wire x1="68.538546875" y1="54.79426875" x2="73.29426875" y2="54.79426875" width="1.016" layer="16"/>
+<wire x1="77.00751875" y1="58.50751875" x2="77.00751875" y2="61.730821875" width="1.016" layer="16"/>
+<wire x1="73.29426875" y1="54.79426875" x2="77.00751875" y2="58.50751875" width="1.016" layer="16"/>
 </signal>
 <signal name="N$18">
 <contactref element="PZEM004T1" pad="N1"/>
 <contactref element="TB7.4" pad="T1"/>
-<wire x1="75.40751875" y1="64.230821875" x2="75.40751875" y2="74.12070625" width="1.016" layer="16"/>
-<wire x1="75.40751875" y1="74.12070625" x2="73.097396875" y2="76.430828125" width="1.016" layer="16"/>
+<wire x1="77.00751875" y1="69.330821875" x2="76.741321875" y2="72.786903125" width="1.016" layer="16"/>
+<wire x1="76.741321875" y1="72.786903125" x2="73.097396875" y2="76.430828125" width="1.016" layer="16"/>
 <wire x1="73.097396875" y1="76.430828125" x2="65.570665625" y2="76.430828125" width="1.016" layer="16"/>
 <wire x1="63.894903125" y1="74.755065625" x2="63.894903125" y2="72.78418125" width="1.016" layer="16"/>
@@
 <wire x1="22.931240625" y1="32.6" x2="32.5959875" y2="22.935253125" width="1.27" layer="16"/>
 <wire x1="32.5959875" y1="22.935253125" x2="61.167328125" y2="22.935253125" width="1.27" layer="16"/>
-<wire x1="74.584809375" y1="36.352734375" x2="75.33924375" y2="36.352734375" width="1.27" layer="16"/>
-<wire x1="61.167328125" y1="22.935253125" x2="74.584809375" y2="36.352734375" width="1.27" layer="16"/>
+<wire x1="72.55408125" y1="34.32200625" x2="76.93924375" y2="34.452734375" width="1.27" layer="16"/>
+<wire x1="61.167328125" y1="22.935253125" x2="72.55408125" y2="34.32200625" width="1.27" layer="16"/>
 </signal>
 <signal name="N$12">
@@
 <contactref element="FUSE-KOTAK1" pad="1"/>
 <contactref element="TB7.1" pad="T2"/>
-<wire x1="75.324909375" y1="14.760603125" x2="75.229090625" y2="14.664784375" width="1.27" layer="16"/>
-<wire x1="75.229090625" y1="14.664784375" x2="75.229090625" y2="9.5067375" width="1.27" layer="16"/>
+<wire x1="76.924909375" y1="9.360603125" x2="76.924909375" y2="1.68908125" width="1.27" layer="16"/>
+<wire x1="76.924909375" y1="1.68908125" x2="76.0067375" y2="0.770909375" width="1.27" layer="16"/>
 </signal>
 </signals>

Commit message: revisi tanggal 07/01/2023
Parts:
- removed RTC1: (no value), rtc3231:RTC3231
- moved C13 3.64 mm to (48.0, 50.6)
Connections:
- net 3V3: no longer RTC1.VCC
- net GND: no longer RTC1.GND
- net SCL: no longer RTC1.SCL
- net SDA: no longer RTC1.SDA
Routing:
- net SDA: track 22.8 -> 0.00 mm
- net 3V3: track 182.7 -> 163.4 mm, vias 7 -> 6
- net SCL: track 17.0 -> 0.00 mm
- net N$1: track 73.4 -> 83.3 mm
- net GND: track 451.7 -> 444.6 mm
- net N$9: track 77.0 -> 79.3 mm
- net N$2: track 74.9 -> 73.0 mm
- net N$13: track 101.1 -> 102.9 mm
- net N$10: track 70.7 -> 72.4 mm
- net N$104: track 109.5 -> 108.2 mm
- net N$15: track 43.5 -> 44.6 mm
- net N$17: track 35.2 -> 34.4 mm
Other:
- board size 80 x 102 mm -> 81 x 98 mm

Commit message: revisi tanggal 08/01/2023
Other:
- board size 81 x 98 mm -> 80 x 102 mm
Changed lines of the file:
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@@
 <board>
 <plain>
-<wire x1="0" y1="89" x2="-1" y2="-9" width="0" layer="20"/>
-<wire x1="-1" y1="-9" x2="80" y2="-9" width="0" layer="20"/>
-<wire x1="80" y1="-9" x2="80" y2="89" width="0" layer="20"/>
-<wire x1="80" y1="89" x2="0" y2="89" width="0" layer="20"/>
+<wire x1="0" y1="91" x2="0" y2="-11" width="0" layer="20"/>
+<wire x1="0" y1="-11" x2="80" y2="-11" width="0" layer="20"/>
+<wire x1="80" y1="-11" x2="80" y2="91" width="0" layer="20"/>
+<wire x1="80" y1="91" x2="0" y2="91" width="0" layer="20"/>
 <text x="72.91520625" y="45.303959375" size="1.4224" layer="25" rot="R90">AC</text>
 <text x="72.972259375" y="59.054909375" size="1.4224" layer="25" rot="R90">CT</text>
@@
 <circle x="11.6" y="87" radius="1.75" width="0.1524" layer="20"/>
 <circle x="63.2" y="-7" radius="1.75" width="0.1524" layer="20"/>
+<dimension x1="-1" y1="-11" x2="-1" y2="91" x3="-5" y3="40" textsize="1.778" layer="1"/>
+<dimension x1="0" y1="-11" x2="80" y2="-11" x3="40" y3="-14" textsize="1.778" layer="1"/>
 </plain>
 <attributes>
