File: revisi/1phasa/untitled.sch (EAGLE design)
At the start: 54 parts, among them J1 U.FL-R-SMT(01), J2 10118193-0001LF, K2 SRD-05VDC-SL-C, Q1 S9013, Q16 MMBT3904, Q17 MMBT3904, Q18 12MHz, U1 AMS1117, U19 CH340G, U2 PC817X2NIP0F, U3 ESP32-WROOM-32D

Commit message: menambahkan fuse
Parts:
- added FUSE-KOTAK1: (no value), FUSE-KOTAK:FUSE-KOTAK
Connections:
- new net N$14: FUSE-KOTAK1.1, TB7.1.T2
- net N$1: now also FUSE-KOTAK1.2; no longer TB7.1.T2
Changed lines of the file:
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@@
 <part name="U3" library="ESP32-WROOM-32D" deviceset="ESP32-WROOM-32D" device=""/>
 <part name="GND10" library="supply1" library_urn="urn:adsk.eagle:library:371" deviceset="GND" device=""/>
+<part name="FUSE-KOTAK1" library="FUSE-KOTAK" deviceset="FUSE-KOTAK" device=""/>
 </parts>
 <sheets>
@@
 <attribute name="VALUE" x="45.21368125" y="194.31315" size="1.77946875" layer="96" rot="R180"/>
 </instance>
-<instance part="TB7.1" gate="G$1" x="129.54" y="254" smashed="yes" rot="R90"/>
+<instance part="TB7.1" gate="G$1" x="124.46" y="254" smashed="yes" rot="R90"/>
 <instance part="TB7.2" gate="G$1" x="134.62" y="190.5" smashed="yes" rot="R270"/>
 <instance part="PZEM004T1" gate="G$1" x="193.04" y="205.74" smashed="yes"/>
@@
 <attribute name="VALUE" x="228.6" y="314.96" size="1.778" layer="96"/>
 </instance>
+<instance part="FUSE-KOTAK1" gate="G$1" x="139.7" y="274.32" smashed="yes" rot="R90"/>
 </instances>
 <busses>
@@
 <pinref part="C12" gate="G$1" pin="P"/>
 <wire x1="147.32" y1="259.08" x2="142.24" y2="259.08" width="0.1524" layer="91"/>
-<pinref part="TB7.1" gate="G$1" pin="T2"/>
-<wire x1="142.24" y1="259.08" x2="137.16" y2="259.08" width="0.1524" layer="91"/>
-<wire x1="137.16" y1="259.08" x2="137.16" y2="256.54" width="0.1524" layer="91"/>
+<pinref part="FUSE-KOTAK1" gate="G$1" pin="2"/>
+<wire x1="142.24" y1="259.08" x2="139.7" y2="259.08" width="0.1524" layer="91"/>
+<wire x1="139.7" y1="259.08" x2="139.7" y2="261.62" width="0.1524" layer="91"/>
 <junction x="142.24" y="259.08"/>
 </segment>
@@
 <junction x="142.24" y="251.46"/>
 <pinref part="TB7.1" gate="G$1" pin="T1"/>
-<wire x1="142.24" y1="251.46" x2="137.16" y2="251.46" width="0.1524" layer="91"/>
+<wire x1="142.24" y1="251.46" x2="132.08" y2="251.46" width="0.1524" layer="91"/>
 </segment>
 </net>
@@
 </segment>
 </net>
+<net name="N$14" class="0">
+<segment>
+<pinref part="FUSE-KOTAK1" gate="G$1" pin="1"/>
+<pinref part="TB7.1" gate="G$1" pin="T2"/>
+<wire x1="137.16" y1="261.62" x2="132.08" y2="261.62" width="0.1524" layer="91"/>
+<wire x1="132.08" y1="261.62" x2="132.08" y2="256.54" width="0.1524" layer="91"/>
+</segment>
+</net>

Commit message: revisi besar-besaran
Connections:
- net RX_PZEM: now also U3.IO17; no longer U3.IO16
- net TX_PZEM: now also U3.IO16; no longer U3.IO17
Changed lines of the file:
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@@
 </segment>
 <segment>
-<pinref part="U3" gate="G$1" pin="IO16"/>
-<wire x1="228.6" y1="353.06" x2="231.14" y2="353.06" width="0.1524" layer="91"/>
-<label x="231.14" y="353.06" size="0.8128" layer="95" xref="yes"/>
+<pinref part="U3" gate="G$1" pin="IO17"/>
+<wire x1="228.6" y1="350.52" x2="231.14" y2="350.52" width="0.1524" layer="91"/>
+<label x="231.14" y="350.52" size="0.8128" layer="95" xref="yes"/>
 </segment>
 </net>
@@
 </segment>
 <segment>
-<pinref part="U3" gate="G$1" pin="IO17"/>
-<wire x1="228.6" y1="350.52" x2="231.14" y2="350.52" width="0.1524" layer="91"/>
-<label x="231.14" y="350.52" size="0.8128" layer="95" xref="yes"/>
+<pinref part="U3" gate="G$1" pin="IO16"/>
+<wire x1="228.6" y1="353.06" x2="231.14" y2="353.06" width="0.1524" layer="91"/>
+<label x="231.14" y="353.06" size="0.8128" layer="95" xref="yes"/>
 </segment>
 </net>

Commit message: revisi tanggal 07/01/2023
Parts:
- removed RTC1: (no value), rtc3231:RTC3231
Connections:
- net 3V3: no longer RTC1.VCC
- net GND: no longer RTC1.GND
- net SCL: no longer RTC1.SCL
- net SDA: no longer RTC1.SDA
Changed lines of the file:
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@@
 <part name="MINI1" library="mini360" deviceset="MINI360" device=""/>
 <part name="SIM800L1" library="sim800l" deviceset="SIM800L" device=""/>
-<part name="RTC1" library="rtc3231" deviceset="RTC3231" device=""/>
 <part name="C13" library="rcl" library_urn="urn:adsk.eagle:library:334" deviceset="C-EU" device="C0805K" package3d_urn="urn:adsk.eagle:package:23681/2" value="10uF"/>
 <part name="P+1" library="supply1" library_urn="urn:adsk.eagle:library:371" deviceset="VCC" device=""/>
 <part name="GND1" library="supply1" library_urn="urn:adsk.eagle:library:371" deviceset="GND" device=""/>
-<part name="GND9" library="supply1" library_urn="urn:adsk.eagle:library:371" deviceset="GND" device=""/>
 <part name="U3" library="ESP32-WROOM-32D" deviceset="ESP32-WROOM-32D" device=""/>
 <part name="GND10" library="supply1" library_urn="urn:adsk.eagle:library:371" deviceset="GND" device=""/>
@@
 <instance part="MINI1" gate="G$1" x="195.58" y="182.88" smashed="yes" rot="R180"/>
 <instance part="SIM800L1" gate="G$1" x="187.96" y="162.56" smashed="yes"/>
-<instance part="RTC1" gate="G$1" x="129.54" y="160.02" smashed="yes"/>
 <instance part="C13" gate="G$1" x="175.26" y="180.34" smashed="yes" rot="R180">
 <attribute name="NAME" x="173.736" y="179.959" size="1.778" layer="95" rot="R180"/>
@@
 <instance part="GND1" gate="1" x="175.26" y="152.4" smashed="yes">
 <attribute name="VALUE" x="172.72" y="149.86" size="1.778" layer="96"/>
-</instance>
-<instance part="GND9" gate="1" x="111.76" y="165.1" smashed="yes">
-<attribute name="VALUE" x="109.22" y="162.56" size="1.778" layer="96"/>
 </instance>
 <instance part="U3" gate="G$1" x="208.28" y="350.52" smashed="yes">
@@
 </segment>
 <segment>
-<pinref part="RTC1" gate="G$1" pin="GND"/>
-<pinref part="GND9" gate="1" pin="GND"/>
-<wire x1="119.38" y1="167.64" x2="111.76" y2="167.64" width="0.1524" layer="91"/>
-</segment>
-<segment>
 <pinref part="U3" gate="G$1" pin="GND"/>
 <pinref part="GND10" gate="1" pin="GND"/>
@@
 </segment>
 <segment>
-<pinref part="RTC1" gate="G$1" pin="VCC"/>
-<wire x1="119.38" y1="165.1" x2="116.84" y2="165.1" width="0.1524" layer="91"/>
-<label x="116.84" y="165.1" size="0.8128" layer="95" rot="R180" xref="yes"/>
-</segment>
-<segment>
 <pinref part="U3" gate="G$1" pin="3V3"/>
 <wire x1="228.6" y1="378.46" x2="231.14" y2="378.46" width="0.1524" layer="91"/>
@@
 <net name="SCL" class="0">
 <segment>
-<pinref part="RTC1" gate="G$1" pin="SCL"/>
-<wire x1="119.38" y1="160.02" x2="116.84" y2="160.02" width="0.1524" layer="91"/>
-<label x="116.84" y="160.02" size="0.8128" layer="95" rot="R180" xref="yes"/>
-</segment>
-<segment>
 <pinref part="U3" gate="G$1" pin="IO22"/>
 <wire x1="228.6" y1="340.36" x2="231.14" y2="340.36" width="0.1524" layer="91"/>
@@
 <net name="SDA" class="0">
 <segment>
-<pinref part="RTC1" gate="G$1" pin="SDA"/>
-<wire x1="119.38" y1="162.56" x2="116.84" y2="162.56" width="0.1524" layer="91"/>
-<label x="116.84" y="162.56" size="0.8128" layer="95" rot="R180" xref="yes"/>
-</segment>
-<segment>
 <pinref part="U3" gate="G$1" pin="IO21"/>

Commit message: revisi PCB jalur, relay, pzem V dan power 1
Parts:
- removed C12: UPM2E100MHD1TO, UPM2E100MHD1TO:UPM2E100MHD1TO
- removed K2: SRD-05VDC-SL-C, SRD-05VDC-SL-C:SRD-05VDC-SL-C
- removed TB7.1: (no value), TB7.62:TB7.62
- added K1: SLA-05VDC-SL-C, SLA-05VDC-SL-C:SLA-05VDC-SL-C
Connections:
- removed net N$15: PZEM004T1.CT+, TB7.3.T2
- removed net N$16: PZEM004T1.CT-, TB7.3.T1
- removed net N$9: K2.COM, TB7.2.T2
- new net N$19: K1.NO, TB7.2.T1
- net N$1: no longer C12.P
- net N$10: now also K1.COM_1, TB7.2.T2; no longer K2.NO, TB7.2.T1
- net N$14: now also PZEM004T1.CT-, TB7.3.T1; no longer TB7.1.T2
- net N$2: now also PZEM004T1.CT+, TB7.3.T2; no longer C12.N, TB7.1.T1
- net N$7: now also K1.COIL_2; no longer K2.A2
- net VCC: now also K1.COIL_1; no longer K2.A1
Changed lines of the file:
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@@
 <part name="C11" library="rcl" library_urn="urn:adsk.eagle:library:334" deviceset="C-EU" device="C0805K" package3d_urn="urn:adsk.eagle:package:23681/2" value="10uF"/>
 <part name="PS1" library="HLK-5M05" deviceset="HLK-5M05" device=""/>
-<part name="C12" library="UPM2E100MHD1TO" deviceset="UPM2E100MHD1TO" device=""/>
 <part name="D1" library="1N5819HW-7" deviceset="1N5819HW-7" device=""/>
 <part name="D2" library="1N5819HW-7" deviceset="1N5819HW-7" device=""/>
@@
 <part name="P+4" library="supply1" library_urn="urn:adsk.eagle:library:371" deviceset="VCC" device=""/>
 <part name="D4" library="SML-LXT0805IW-TR" deviceset="SML-LXT0805IW-TR" device=""/>
-<part name="TB7.1" library="TB7.62" deviceset="TB7.62" device=""/>
 <part name="TB7.2" library="TB7.62" deviceset="TB7.62" device=""/>
 <part name="PZEM004T1" library="PZEM004T" deviceset="PZEM004T" device=""/>
@@
 <part name="TB7.3" library="TB7.62" deviceset="TB7.62" device=""/>
 <part name="TB7.4" library="TB7.62" deviceset="TB7.62" device=""/>
-<part name="K2" library="SRD-05VDC-SL-C" deviceset="SRD-05VDC-SL-C" device=""/>
 <part name="D5" library="SML-LXT0805IW-TR" deviceset="SML-LXT0805IW-TR" device=""/>
 <part name="R3" library="rcl" library_urn="urn:adsk.eagle:library:334" deviceset="R-EU_" device="R0805" package3d_urn="urn:adsk.eagle:package:23553/2" value="10k"/>
@@
 <part name="GND10" library="supply1" library_urn="urn:adsk.eagle:library:371" deviceset="GND" device=""/>
 <part name="FUSE-KOTAK1" library="FUSE-KOTAK" deviceset="FUSE-KOTAK" device=""/>
+<part name="K1" library="SLA-05VDC-SL-C" deviceset="SLA-05VDC-SL-C" device=""/>
 </parts>
 <sheets>
@@
 <attribute name="VALUE" x="152.4" y="248.92" size="1.778" layer="96"/>
 </instance>
-<instance part="C12" gate="G$1" x="142.24" y="256.54" smashed="yes" rot="R270">
-<attribute name="NAME" x="146.05" y="259.08" size="1.778" layer="95" rot="R270"/>
-</instance>
 <instance part="D1" gate="G$1" x="187.96" y="259.08" smashed="yes">
 <attribute name="NAME" x="182.88" y="261.62" size="1.778" layer="95"/>
@@
 <attribute name="VALUE" x="45.21368125" y="194.31315" size="1.77946875" layer="96" rot="R180"/>
 </instance>
-<instance part="TB7.1" gate="G$1" x="124.46" y="254" smashed="yes" rot="R90"/>
-<instance part="TB7.2" gate="G$1" x="134.62" y="190.5" smashed="yes" rot="R270"/>
+<instance part="TB7.2" gate="G$1" x="144.78" y="190.5" smashed="yes" rot="R270"/>
 <instance part="PZEM004T1" gate="G$1" x="193.04" y="205.74" smashed="yes"/>
 <instance part="GND6" gate="1" x="218.44" y="205.74" smashed="yes">
@@
 <instance part="TB7.3" gate="G$1" x="170.18" y="218.44" smashed="yes"/>
 <instance part="TB7.4" gate="G$1" x="157.48" y="218.44" smashed="yes"/>
-<instance part="K2" gate="G$1" x="101.6" y="187.96" smashed="yes">
-<attribute name="NAME" x="96.5191" y="193.803040625" size="1.77831875" layer="95"/>
-<attribute name="VALUE" x="96.516809375" y="177.7936" size="1.77911875" layer="96"/>
-</instance>
 <instance part="D5" gate="G$1" x="71.12" y="279.4" smashed="yes" rot="R90">
 <attribute name="NAME" x="67.04973125" y="277.36486875" size="1.780740625" layer="95" rot="R90"/>
@@
 </instance>
 <instance part="FUSE-KOTAK1" gate="G$1" x="139.7" y="274.32" smashed="yes" rot="R90"/>
+<instance part="K1" gate="G$1" x="129.54" y="187.96" smashed="yes" rot="R180">
+<attribute name="NAME" x="100.33" y="180.34" size="1.778" layer="95" rot="R180" align="center-left"/>
+<attribute name="VALUE" x="100.33" y="182.88" size="1.778" layer="96" rot="R180" align="center-left"/>
+</instance>
 </instances>
 <busses>
@@
 <pinref part="P+4" gate="VCC" pin="VCC"/>
 <junction x="73.66" y="205.74"/>
-<pinref part="K2" gate="G$1" pin="A1"/>
-<wire x1="93.98" y1="190.5" x2="93.98" y2="195.58" width="0.1524" layer="91"/>
 <wire x1="93.98" y1="195.58" x2="86.36" y2="195.58" width="0.1524" layer="91"/>
 <junction x="86.36" y="195.58"/>
+<pinref part="K1" gate="G$1" pin="COIL_1"/>
+<wire x1="96.52" y1="190.5" x2="93.98" y2="190.5" width="0.1524" layer="91"/>
+<wire x1="93.98" y1="190.5" x2="93.98" y2="195.58" width="0.1524" layer="91"/>
 </segment>
 <segment>
@@
 <segment>
 <pinref part="PS1" gate="G$1" pin="AC1"/>
-<pinref part="C12" gate="G$1" pin="P"/>
-<wire x1="147.32" y1="259.08" x2="142.24" y2="259.08" width="0.1524" layer="91"/>
+<wire x1="147.32" y1="259.08" x2="139.7" y2="259.08" width="0.1524" layer="91"/>
 <pinref part="FUSE-KOTAK1" gate="G$1" pin="2"/>
-<wire x1="142.24" y1="259.08" x2="139.7" y2="259.08" width="0.1524" layer="91"/>
 <wire x1="139.7" y1="259.08" x2="139.7" y2="261.62" width="0.1524" layer="91"/>
-<junction x="142.24" y="259.08"/>
 </segment>
 </net>
@@
 <segment>
 <pinref part="PS1" gate="G$1" pin="AC2"/>
-<pinref part="C12" gate="G$1" pin="N"/>
 <wire x1="147.32" y1="254" x2="147.32" y2="251.46" width="0.1524" layer="91"/>
-<wire x1="147.32" y1="251.46" x2="142.24" y2="251.46" width="0.1524" layer="91"/>
-<junction x="142.24" y="251.46"/>
-<pinref part="TB7.1" gate="G$1" pin="T1"/>
-<wire x1="142.24" y1="251.46" x2="132.08" y2="251.46" width="0.1524" layer="91"/>
+<wire x1="147.32" y1="251.46" x2="132.08" y2="251.46" width="0.1524" layer="91"/>
+<wire x1="132.08" y1="251.46" x2="132.08" y2="228.6" width="0.1524" layer="91"/>
+<wire x1="132.08" y1="228.6" x2="172.72" y2="228.6" width="0.1524" layer="91"/>
+<pinref part="PZEM004T1" gate="G$1" pin="CT+"/>
+<pinref part="TB7.3" gate="G$1" pin="T2"/>
+<wire x1="182.88" y1="208.28" x2="172.72" y2="208.28" width="0.1524" layer="91"/>
+<wire x1="172.72" y1="208.28" x2="172.72" y2="210.82" width="0.1524" layer="91"/>
+<wire x1="172.72" y1="228.6" x2="172.72" y2="210.82" width="0.1524" layer="91"/>
+<junction x="172.72" y="210.82"/>
 </segment>
 </net>
@@
 <pinref part="Q1" gate="G$1" pin="C"/>
 <wire x1="86.36" y1="182.88" x2="86.36" y2="180.34" width="0.1524" layer="91"/>
-<pinref part="K2" gate="G$1" pin="A2"/>
 <wire x1="86.36" y1="180.34" x2="86.36" y2="177.8" width="0.1524" layer="91"/>
-<wire x1="93.98" y1="182.88" x2="93.98" y2="180.34" width="0.1524" layer="91"/>
-<wire x1="93.98" y1="180.34" x2="86.36" y2="180.34" width="0.1524" layer="91"/>
 <junction x="86.36" y="180.34"/>
+<pinref part="K1" gate="G$1" pin="COIL_2"/>
+<wire x1="96.52" y1="193.04" x2="101.6" y2="193.04" width="0.1524" layer="91"/>
+<wire x1="101.6" y1="193.04" x2="101.6" y2="180.34" width="0.1524" layer="91"/>
+<wire x1="101.6" y1="180.34" x2="86.36" y2="180.34" width="0.1524" layer="91"/>
 </segment>
 </net>
@@
 </segment>
 </net>
-<net name="N$9" class="0">
-<segment>
-<pinref part="TB7.2" gate="G$1" pin="T2"/>
-<wire x1="127" y1="187.96" x2="127" y2="182.88" width="0.1524" layer="91"/>
-<wire x1="127" y1="182.88" x2="114.3" y2="182.88" width="0.1524" layer="91"/>
-<wire x1="114.3" y1="182.88" x2="114.3" y2="187.96" width="0.1524" layer="91"/>
-<pinref part="K2" gate="G$1" pin="COM"/>
-<wire x1="114.3" y1="187.96" x2="109.22" y2="187.96" width="0.1524" layer="91"/>
-</segment>
-</net>
 <net name="N$4" class="0">
 <segment>
@@
 <wire x1="228.6" y1="353.06" x2="231.14" y2="353.06" width="0.1524" layer="91"/>
 <label x="231.14" y="353.06" size="0.8128" layer="95" xref="yes"/>
-</segment>
-</net>
-<net name="N$15" class="0">
-<segment>
-<pinref part="PZEM004T1" gate="G$1" pin="CT+"/>
-<pinref part="TB7.3" gate="G$1" pin="T2"/>
-<wire x1="182.88" y1="208.28" x2="172.72" y2="208.28" width="0.1524" layer="91"/>
-<wire x1="172.72" y1="208.28" x2="172.72" y2="210.82" width="0.1524" layer="91"/>
-</segment>
-</net>
-<net name="N$16" class="0">
-<segment>
-<pinref part="PZEM004T1" gate="G$1" pin="CT-"/>
-<pinref part="TB7.3" gate="G$1" pin="T1"/>
-<wire x1="182.88" y1="205.74" x2="167.64" y2="205.74" width="0.1524" layer="91"/>
-<wire x1="167.64" y1="205.74" x2="167.64" y2="210.82" width="0.1524" layer="91"/>
 </segment>
 </net>
@@
 <pinref part="R42" gate="G$1" pin="2"/>
 <wire x1="147.32" y1="353.06" x2="144.78" y2="353.06" width="0.1524" layer="91"/>
-</segment>
-</net>
-<net name="N$10" class="0">
-<segment>
-<pinref part="TB7.2" gate="G$1" pin="T1"/>
-<pinref part="K2" gate="G$1" pin="NO"/>
-<wire x1="127" y1="193.04" x2="109.22" y2="193.04" width="0.1524" layer="91"/>
-<wire x1="109.22" y1="193.04" x2="109.22" y2="190.5" width="0.1524" layer="91"/>
 </segment>
 </net>
@@
 <segment>
 <pinref part="FUSE-KOTAK1" gate="G$1" pin="1"/>
-<pinref part="TB7.1" gate="G$1" pin="T2"/>
 <wire x1="137.16" y1="261.62" x2="132.08" y2="261.62" width="0.1524" layer="91"/>
 <wire x1="132.08" y1="261.62" x2="132.08" y2="256.54" width="0.1524" layer="91"/>
-</segment>
-</net>
+<wire x1="132.08" y1="256.54" x2="127" y2="256.54" width="0.1524" layer="91"/>
+<wire x1="127" y1="256.54" x2="127" y2="223.52" width="0.1524" layer="91"/>
+<pinref part="PZEM004T1" gate="G$1" pin="CT-"/>
+<pinref part="TB7.3" gate="G$1" pin="T1"/>
+<wire x1="182.88" y1="205.74" x2="167.64" y2="205.74" width="0.1524" layer="91"/>
+<wire x1="167.64" y1="205.74" x2="167.64" y2="210.82" width="0.1524" layer="91"/>
+<wire x1="127" y1="223.52" x2="167.64" y2="223.52" width="0.1524" layer="91"/>
+<wire x1="167.64" y1="223.52" x2="167.64" y2="210.82" width="0.1524" layer="91"/>
+<junction x="167.64" y="210.82"/>
+</segment>
+</net>
+<net name="N$10" class="0">
+<segment>
+<pinref part="K1" gate="G$1" pin="COM_1"/>
+<pinref part="TB7.2" gate="G$1" pin="T2"/>
+<wire x1="129.54" y1="187.96" x2="137.16" y2="187.96" width="0.1524" layer="91"/>
+</segment>
+</net>
+<net name="N$19" class="0">
+<segment>
+<pinref part="K1" gate="G$1" pin="NO"/>
+<pinref part="TB7.2" gate="G$1" pin="T1"/>
+<wire x1="129.54" y1="193.04" x2="137.16" y2="193.04" width="0.1524" layer="91"/>
+</segment>
+</net>

Commit message: fix
Parts:
- R2, R3, R47: value 10k -> 1k
Changed lines of the file:
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@@
 <part name="R46" library="rcl" library_urn="urn:adsk.eagle:library:334" deviceset="R-EU_" device="R0805" package3d_urn="urn:adsk.eagle:package:23553/2" value="10k"/>
 <part name="D20" library="SML-LXT0805IW-TR" deviceset="SML-LXT0805IW-TR" device=""/>
-<part name="R47" library="rcl" library_urn="urn:adsk.eagle:library:334" deviceset="R-EU_" device="R0805" package3d_urn="urn:adsk.eagle:package:23553/2" value="10k"/>
+<part name="R47" library="rcl" library_urn="urn:adsk.eagle:library:334" deviceset="R-EU_" device="R0805" package3d_urn="urn:adsk.eagle:package:23553/2" value="1k"/>
 <part name="P+5" library="supply1" library_urn="urn:adsk.eagle:library:371" deviceset="VCC" device=""/>
 <part name="C11" library="rcl" library_urn="urn:adsk.eagle:library:334" deviceset="C-EU" device="C0805K" package3d_urn="urn:adsk.eagle:package:23681/2" value="10uF"/>
@@
 <part name="R1" library="rcl" library_urn="urn:adsk.eagle:library:334" deviceset="R-EU_" device="R0805" package3d_urn="urn:adsk.eagle:package:23553/2" value="330"/>
 <part name="U2" library="PC817X2NIP0F" deviceset="PC817X2NIP0F" device=""/>
-<part name="R2" library="rcl" library_urn="urn:adsk.eagle:library:334" deviceset="R-EU_" device="R0805" package3d_urn="urn:adsk.eagle:package:23553/2" value="10k"/>
+<part name="R2" library="rcl" library_urn="urn:adsk.eagle:library:334" deviceset="R-EU_" device="R0805" package3d_urn="urn:adsk.eagle:package:23553/2" value="1k"/>
 <part name="D3" library="US1M-13" deviceset="US1M-13" device=""/>
 <part name="Q1" library="S9013" deviceset="S9013" device=""/>
@@
 <part name="TB7.4" library="TB7.62" deviceset="TB7.62" device=""/>
 <part name="D5" library="SML-LXT0805IW-TR" deviceset="SML-LXT0805IW-TR" device=""/>
-<part name="R3" library="rcl" library_urn="urn:adsk.eagle:library:334" deviceset="R-EU_" device="R0805" package3d_urn="urn:adsk.eagle:package:23553/2" value="10k"/>
+<part name="R3" library="rcl" library_urn="urn:adsk.eagle:library:334" deviceset="R-EU_" device="R0805" package3d_urn="urn:adsk.eagle:package:23553/2" value="1k"/>
 <part name="MINI1" library="mini360" deviceset="MINI360" device=""/>
 <part name="SIM800L1" library="sim800l" deviceset="SIM800L" device=""/>
