File: revisi/3phasa/untitled.sch (EAGLE design)
At the start: 59 parts, among them J1 U.FL-R-SMT(01), J2 10118193-0001LF, K2 SRD-05VDC-SL-C, Q1 S9013, Q16 MMBT3904, Q17 MMBT3904, Q18 12MHz, U1 AMS1117, U19 CH340G, U2 PC817X2NIP0F, U3 ESP32-WROOM-32D

Commit message: revisi besar-besaran
Parts:
- added D10, D11, D12, D6, D8: US1M-13, US1M-13:US1M-13
- added D7, D9: SML-LXT0805IW-TR, SML-LXT0805IW-TR:SML-LXT0805IW-TR
- added K1, K3: SRD-05VDC-SL-C, SRD-05VDC-SL-C:SRD-05VDC-SL-C
- added Q2, Q3: S9013, S9013:S9013
- added R4, R6: 330, rcl:R-EU_R0805
- added R5, R7, R8: 10k, rcl:R-EU_R0805
- added TB7.10, TB7.9: (no value), TB7.62:TB7.62
- added U4, U5: PC817X2NIP0F, PC817X2NIP0F:PC817X2NIP0F
Connections:
- new net N$26: R5.1, U4.CT
- new net N$27: Q2.B, U4.ET
- new net N$28: D6.A, K1.A2, Q2.C
- new net N$29: K1.COM, TB7.9.T1
- new net N$30: D7.C, U4.A
- new net N$31: D7.A, R4.2
- new net N$32: K1.NO, TB7.9.T2
- new net N$33: R7.1, U5.CT
- new net N$34: Q3.B, U5.ET
- new net N$35: D8.A, K3.A2, Q3.C
- new net N$36: K3.COM, TB7.10.T1
- new net N$37: D9.C, U5.A
- new net N$38: D9.A, R6.2
- new net N$39: K3.NO, TB7.10.T2
- new net N$40: D10.K, PZEM004T1.TX
- new net N$41: D11.K, PZEM004T2.TX
- new net N$42: D12.K, PZEM004T3.TX
- new net RELAY1: R4.1, U3.IO33
- new net RELAY2: R6.1, U3.IO27
- net GND: now also Q2.E, Q3.E, U4.C, U5.C
- net RX_PZEM: now also U3.IO17; no longer U3.IO16
- net TX_PZEM: now also D10.A, D11.A, D12.A, R8.1, U3.IO16; no longer PZEM004T1.TX, PZEM004T2.TX, PZEM004T3.TX, U3.IO17
- net VCC: now also D6.K, D8.K, K1.A1, K3.A1, R5.2, R7.2, R8.2
